Commit message: Added mesh file with origin exported at base_link for correct visualization

File: urdf/swd_starter_kit.urdf (robot description, URDF)
Before this commit: robot swd_starter_kit, 4 links, 3 joints
Links:
- added link base_footprint_link
- link base_link: geometry collision mesh filename=package://arav_visualization/assets/arav_assembly_v3_origin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 scale=0.001 0.001 0.001; visual mesh filename=package://arav_visualization/assets/arav_assembly_v3_origin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 scale=0.001 0.001 0.001
Joints:
- added joint base_joint: type fixed, parent base_footprint_link, child base_link, origin xyz=0.0 0.0 0.1365 rpy= 0 0 0 
